File: OCP2PCIe-H-F-4/OCP2PCIe-H-F-4-V3.0Beta/V1.kicad_pcb (KiCad board)
At the start: 2 copper layers, 112.1 x 78.2 mm, 30 parts, among them J1 PCIe_x8, J2 Conn_02x40_Top_Bottom, J3 Conn_01x02, J4 Conn_01x02, U1 DM02, U2 9DBL411B

Commit message: tuning clock
Connections:
- R5 pad 2: GND -> +3V3
Routing:
- net +3V3: track 100.3 -> 107.6 mm
