File: OCP2PCIe-H-F-4/OCP2PCIe-H-F-4-V3.0Beta/V1.sch (KiCad schematic (older format))
At the start: 24 parts, among them J1 PCIe_x8, J2 Conn_02x40_Top_Bottom, J3 Conn_01x02, J4 Conn_01x02, U1 DM02, U2 9DBL411B

Commit message: fixed
Parts:
- R1: value R -> 34.46
Changed lines of the file:
@@
 P 10300 4350
 F 0 "R1" V 10200 4350 50  0000 C CNN
-F 1 "R" V 10200 4450 50  0000 C CNN
+F 1 "34.46" V 10200 4550 50  0000 C CNN
 F 2 "Resistor_SMD:R_0402_1005Metric_Pad0.72x0.64mm_HandSolder" V 10230 4350 50  0001 C CNN
 F 3 "~" H 10300 4350 50  0001 C CNN

Commit message: tuning pcie lane
Parts:
- added R5: 100ohm, Resistor_SMD:R_0603_1608Metric_Pad0.98x0.95mm_HandSolder, symbol Device:R
Connections:
- wire segments 81 -> 83
Changed lines of the file:
@@
 REFCLK-
 Text GLabel 7950 4600 0    50   Input ~ 0
-OE1
+OE0
 Text GLabel 10450 5600 1    50   Input ~ 0
 OE0
@@
 OE1
 Text GLabel 9050 5200 2    50   Input ~ 0
-OE0
-$Comp
-L power:GND #PWR0204
-U 1 1 60B6B584
-P 10450 6200
-F 0 "#PWR0204" H 10450 5950 50  0001 C CNN
-F 1 "GND" H 10455 6027 50  0000 C CNN
-F 2 "" H 10450 6200 50  0001 C CNN
-F 3 "" H 10450 6200 50  0001 C CNN
-	1    10450 6200
-	1    0    0    -1
-$EndComp
-$Comp
-L power:GND #PWR0205
-U 1 1 60B6BC15
-P 10650 6200
-F 0 "#PWR0205" H 10650 5950 50  0001 C CNN
-F 1 "GND" H 10655 6027 50  0000 C CNN
-F 2 "" H 10650 6200 50  0001 C CNN
-F 3 "" H 10650 6200 50  0001 C CNN
-	1    10650 6200
-	1    0    0    -1
-$EndComp
+OE1
 Text GLabel 10450 4450 2    50   Input ~ 0
+REFCLK0+
+Text GLabel 10450 4350 2    50   Input ~ 0
+REFCLK0-
+Text GLabel 10450 4850 2    50   Input ~ 0
 REFCLK1+
-Text GLabel 10450 4350 2    50   Input ~ 0
+Text GLabel 10450 4750 2    50   Input ~ 0
 REFCLK1-
-Text GLabel 10450 4850 2    50   Input ~ 0
-REFCLK0+
-Text GLabel 10450 4750 2    50   Input ~ 0
-REFCLK0-
 NoConn ~ 9050 5750
 NoConn ~ 9050 5900
@@
 $EndComp
 Text GLabel 10150 4350 0    50   Input ~ 0
+DIF0_N
+Text GLabel 10150 4450 0    50   Input ~ 0
+DIF0_P
+Text GLabel 9050 4600 2    50   Input ~ 0
+DIF0_N
+Text GLabel 9050 4750 2    50   Input ~ 0
+DIF0_P
+Text GLabel 10150 4750 0    50   Input ~ 0
 DIF1_N
-Text GLabel 10150 4450 0    50   Input ~ 0
+Text GLabel 10150 4850 0    50   Input ~ 0
 DIF1_P
-Text GLabel 9050 4600 2    50   Input ~ 0
+Text GLabel 9050 5300 2    50   Input ~ 0
 DIF1_N
-Text GLabel 9050 4750 2    50   Input ~ 0
+Text GLabel 9050 5450 2    50   Input ~ 0
 DIF1_P
-Text GLabel 10150 4750 0    50   Input ~ 0
-DIF0_N
-Text GLabel 10150 4850 0    50   Input ~ 0
-DIF0_P
-Text GLabel 9050 5300 2    50   Input ~ 0
-DIF0_N
-Text GLabel 9050 5450 2    50   Input ~ 0
-DIF0_P
 NoConn ~ 1750 2850
 NoConn ~ 1750 2950
 NoConn ~ 5450 2950
 NoConn ~ 5450 3050
+$Comp
+L Device:R R5
+U 1 1 60AAEBA0
+P 9900 6200
+F 0 "R5" V 9693 6200 50  0000 C CNN
+F 1 "100ohm" V 9784 6200 50  0000 C CNN
+F 2 "Resistor_SMD:R_0603_1608Metric_Pad0.98x0.95mm_HandSolder" V 9830 6200 50  0001 C CNN
+F 3 "~" H 9900 6200 50  0001 C CNN
+	1    9900 6200
+	0    1    1    0
+$EndComp
+$Comp
+L power:GND #PWR?
+U 1 1 60AAF187
+P 9750 6200
+F 0 "#PWR?" H 9750 5950 50  0001 C CNN
+F 1 "GND" H 9755 6027 50  0000 C CNN
+F 2 "" H 9750 6200 50  0001 C CNN
+F 3 "" H 9750 6200 50  0001 C CNN
+	1    9750 6200
+	0    1    1    0
+$EndComp
+Wire Wire Line
+	10050 6200 10450 6200
+Connection ~ 10450 6200
+Wire Wire Line
+	10450 6200 10650 6200
 $EndSCHEMATC

Commit message: tuning clock
Connections:
- wire segments 83 -> 84
Changed lines of the file:
@@
 NoConn ~ 5450 2950
 NoConn ~ 5450 3050
+Wire Wire Line
+	10050 6200 10450 6200
+Connection ~ 10450 6200
+Wire Wire Line
+	10450 6200 10650 6200
 $Comp
 L Device:R R5
@@
 $EndComp
 $Comp
-L power:GND #PWR?
-U 1 1 60AAF187
-P 9750 6200
-F 0 "#PWR?" H 9750 5950 50  0001 C CNN
-F 1 "GND" H 9755 6027 50  0000 C CNN
-F 2 "" H 9750 6200 50  0001 C CNN
-F 3 "" H 9750 6200 50  0001 C CNN
-	1    9750 6200
-	0    1    1    0
+L power:+3V3 #PWR?
+U 1 1 60BBC1BD
+P 9650 6200
+F 0 "#PWR?" H 9650 6050 50  0001 C CNN
+F 1 "+3V3" H 9665 6373 50  0000 C CNN
+F 2 "" H 9650 6200 50  0001 C CNN
+F 3 "" H 9650 6200 50  0001 C CNN
+	1    9650 6200
+	1    0    0    -1
 $EndComp
 Wire Wire Line
-	10050 6200 10450 6200
-Connection ~ 10450 6200
-Wire Wire Line
-	10450 6200 10650 6200
+	9750 6200 9650 6200
 $EndSCHEMATC
