File: OCP2PCIe-H-F-4/OCP2PCIe-H-F-8-V4.0Beta/V1.kicad_pcb (KiCad board)
At the start: 2 copper layers, 112.1 x 78.2 mm, 15 parts, among them J1 PCIe_x8, J2 Conn_02x40_Top_Bottom, J3 Conn_01x02, J4 Conn_01x02, U1 DM02

Commit message: ast2300 first
Routing:
- net HSI0_N: track 68.4 -> 71.0 mm
- net HSO0_N: track 53.0 -> 55.6 mm
- net GND: vias 109 -> 113
